Commit message: orientation last joint

File: robot_descriptions/ur_robot/ur_description/urdf/ur10.urdf (robot description, URDF)
Before this commit: robot urdf10, 10 links, 9 joints
Joints:
- joint wrist_1_joint: limit lower=-3.141592653589793 upper=3.141592653589793 effort=54.0 velocity=3.2 -> lower=-3.141592653589793 upper=3.141592653589793 effort=150 velocity=3.2
- joint wrist_2_joint: limit lower=-3.141592653589793 upper=3.141592653589793 effort=54.0 velocity=3.2 -> lower=-3.141592653589793 upper=3.141592653589793 effort=150 velocity=3.2
- joint wrist_3_joint: limit lower=-3.141592653589793 upper=3.141592653589793 effort=54.0 velocity=3.2 -> lower=-3.141592653589793 upper=3.141592653589793 effort=150 velocity=3.2

File: src/tum_ics_ur10_robot/tum_ics_ur10_description/urdf/ur10.urdf.xacro (robot description, xacro)
@@ -171,8 +171,8 @@
       <axis xyz="0 1 0" />
       <xacro:unless value="${joint_limited}">
-        <limit lower="${-2.0 * pi}" upper="${2.0 * pi}" effort="54.0" velocity="3.2"/>
-      </xacro:unless>
-      <xacro:if value="${joint_limited}">
-        <limit lower="${-pi}" upper="${pi}" effort="54.0" velocity="3.2"/>
+        <limit lower="${-2.0 * pi}" upper="${2.0 * pi}" effort="200" velocity="3.2"/>
+      </xacro:unless>
+      <xacro:if value="${joint_limited}">
+        <limit lower="${-pi}" upper="${pi}" effort="200" velocity="3.2"/>
       </xacro:if>
       <dynamics damping="0.0" friction="0.0"/>
@@ -202,8 +202,8 @@
       <axis xyz="0 0 1" />
       <xacro:unless value="${joint_limited}">
-        <limit lower="${-2.0 * pi}" upper="${2.0 * pi}" effort="54.0" velocity="3.2"/>
-      </xacro:unless>
-      <xacro:if value="${joint_limited}">
-        <limit lower="${-pi}" upper="${pi}" effort="54.0" velocity="3.2"/>
+        <limit lower="${-2.0 * pi}" upper="${2.0 * pi}" effort="200" velocity="3.2"/>
+      </xacro:unless>
+      <xacro:if value="${joint_limited}">
+        <limit lower="${-pi}" upper="${pi}" effort="200" velocity="3.2"/>
       </xacro:if>
       <dynamics damping="0.0" friction="0.0"/>
@@ -233,8 +233,8 @@
       <axis xyz="0 1 0" />
       <xacro:unless value="${joint_limited}">
-        <limit lower="${-2.0 * pi}" upper="${2.0 * pi}" effort="54.0" velocity="3.2"/>
-      </xacro:unless>
-      <xacro:if value="${joint_limited}">
-        <limit lower="${-pi}" upper="${pi}" effort="54.0" velocity="3.2"/>
+        <limit lower="${-2.0 * pi}" upper="${2.0 * pi}" effort="200" velocity="3.2"/>
+      </xacro:unless>
+      <xacro:if value="${joint_limited}">
+        <limit lower="${-pi}" upper="${pi}" effort="200" velocity="3.2"/>
       </xacro:if>
       <dynamics damping="0.0" friction="0.0"/>
